File: imu-gc.kicad_pcb (KiCad board)
At the start: 2 copper layers, 20 x 30 mm, 21 parts, among them U1 nRF54L15-QFXX, Y1 32Mhz

Commit message: typ l
Parts:
- C10: renamed from C8; footprint Capacitor_SMD:C_0402_1005Metric -> Capacitor_SMD:C_0201_0603Metric
- C11: renamed from C9; footprint Capacitor_SMD:C_0402_1005Metric -> Capacitor_SMD:C_0201_0603Metric
- C12: renamed from C11; footprint Capacitor_SMD:C_0402_1005Metric -> Capacitor_SMD:C_0201_0603Metric
- L2: renamed from L1; footprint Inductor_SMD:L_0402_1005Metric -> Inductor_SMD:L_0201_0603Metric
- L3, L4: footprint Inductor_SMD:L_0402_1005Metric -> Inductor_SMD:L_0201_0603Metric
- moved C7 30.8 mm to (162.6, 123.1)
- moved Y1 4.16 mm to (160.8, 117.3)
- moved C12 1.22 mm to (165.3, 124.0)
- moved L4 0.90 mm to (165.3, 124.8)
- moved C11 0.82 mm to (163.8, 124.0)
- moved L3 0.48 mm to (163.8, 124.8)
- moved C10 0.42 mm to (162.3, 124.0)
- moved L2 0.07 mm to (162.3, 124.8)
- renumbered C7 to C13, C10 to C6, C12 to C7, C13 to C8, C6 to C9, L2 to L1
Routing:
- net Net-(U1-DECA): track 5.04 -> 0.00 mm
- net Net-(U1-XC2): track 3.71 -> 0.00 mm
- net Net-(U1-XC1): track 3.57 -> 0.00 mm
- net Net-(C11-Pad1): track 2.07 -> 0.00 mm
- net Net-(C10-Pad1): track 2.07 -> 0.00 mm
- net GND: track 10.0 -> 9.55 mm, vias 3 -> 2
- added copper zone on F.Cu, net Net-(C10-Pad1)

Commit message: Atennas? RF for sures
Parts:
- moved C12 11.4 mm to (157.5, 115.6)
- moved L4 10.9 mm to (157.9, 116.8), turned to 90 degrees
- moved C11 8.26 mm to (158.2, 117.9), turned to 0 degrees
- moved L3 8.25 mm to (157.9, 119.0), turned to 90 degrees
- moved Y1 7.45 mm to (154.1, 120.5), turned to 0 degrees
- moved C7 6.96 mm to (156.2, 120.3), turned to 90 degrees
- moved C10 6.26 mm to (157.1, 120.5), turned to -90 degrees
- moved L2 6.13 mm to (157.9, 120.5), turned to 90 degrees
- moved U1 1.14 mm to (158.1, 125.7), turned to 90 degrees
Connections:
- C12 pad 1: /RF -> GND
- L4 pad 2: /RF -> GND
Routing:
- net Net-(U1-XC2): track 0.00 -> 3.85 mm
- net Net-(U1-XC1): track 0.00 -> 3.63 mm
- net Net-(U1-DECA): track 0.00 -> 2.32 mm
- net GND: track 9.55 -> 8.18 mm
- net /RF: track 0.90 -> 0.00 mm
- added copper zone on F.Cu, net Net-(C11-Pad1)
Other:
- board size 20 x 30 mm -> 30 x 40 mm

Commit message: bom + readm
Parts:
- moved C6 27.2 mm to (161.6, 122.9), turned to 90 degrees
- moved C7 8.85 mm to (158.6, 128.8), turned to 180 degrees
- moved C11 6.14 mm to (163.7, 120.8)
- moved C12 6.14 mm to (163.0, 118.5)
- moved L2 6.14 mm to (163.3, 123.4)
- moved L3 6.14 mm to (163.3, 121.9)
- moved L4 6.14 mm to (163.3, 119.6)
- moved Y1 6.14 mm to (159.5, 123.4)
- moved C10 6.14 mm to (162.5, 123.4)
- moved U1 6.14 mm to (163.5, 128.5)
Routing:
- net GND: track 8.18 -> 16.4 mm, vias 2 -> 5
- added copper zone on F.Cu, net GND
- removed copper zone on F.Cu, net Net-(C10-Pad1)
- removed copper zone on F.Cu, net Net-(C11-Pad1)
Other:
- board size 30 x 40 mm -> 30 x 39.5 mm

Commit message: bom + readm
Parts:
- moved C2 31.5 mm to (168.1, 127.1)
- moved C1 26.5 mm to (164.9, 133.1), turned to -90 degrees
- moved C3 25.3 mm to (159.3, 125.5), turned to 180 degrees
- moved C4 20.2 mm to (158.9, 130.1), turned to 180 degrees
- moved C5 18.3 mm to (158.9, 131.0), turned to 180 degrees
- moved C7 0.41 mm to (159.0, 128.7)
Routing:
- net /VDD_MCU: track 0.00 -> 6.33 mm
- net GND: track 16.4 -> 20.1 mm, vias 5 -> 11

Commit message: typ finsihed. yeygit add -A
Parts:
- C1, C2, C4, C5: value 1000nF -> 100nF; footprint Capacitor_SMD:C_0402_1005Metric -> Capacitor_SMD:C_0201_0603Metric
- C3: value 1000nF -> 10uF
- C6, C7, C8, C9: footprint Capacitor_SMD:C_0402_1005Metric -> Capacitor_SMD:C_0201_0603Metric
- FB1: footprint Inductor_SMD:L_0402_1005Metric -> Inductor_SMD:L_0201_0603Metric
- L1: footprint Inductor_SMD:L_0402_1005Metric -> Inductor_SMD:L_0603_1608Metric
- R1: footprint Resistor_SMD:R_0402_1005Metric -> Resistor_SMD:R_0201_0603Metric
- moved R1 35.8 mm to (164.1, 124.2), turned to 90 degrees
- moved C13 25.2 mm to (164.9, 124.0), turned to 90 degrees
- moved C8 24.1 mm to (159.2, 127.0), turned to 180 degrees
- moved FB1 22.7 mm to (159.2, 127.7), turned to 180 degrees
- moved L1 22.0 mm to (157.3, 128.8), turned to 90 degrees
- moved C9 18.4 mm to (159.2, 129.9), turned to 180 degrees
- moved C5 9.71 mm to (167.8, 127.2), turned to 0 degrees
- moved C2 9.60 mm to (159.2, 130.7), turned to 180 degrees
- moved C1 9.29 mm to (159.5, 125.5), turned to 180 degrees
- moved C4 6.59 mm to (164.9, 132.9), turned to -90 degrees
- moved C3 6.12 mm to (159.3, 131.6)
- moved C7 0.32 mm to (159.2, 128.4)
Connections:
- C13 pad 2: unconnected-(C13-Pad2) -> GND
Routing:
- net Net-(U1-DECA): track 2.63 -> 12.5 mm, vias 0 -> 2
- net Net-(U1-DECD): track 0.00 -> 3.21 mm
- net Net-(U1-DCC): track 0.00 -> 2.68 mm
- net Net-(U1-~{RESET}): track 0.00 -> 2.08 mm
- net GND: track 20.1 -> 20.3 mm, vias 11 -> 13

Commit message: IMU ok, power startd
Parts:
- added C14: 100nF, Capacitor_SMD:C_0402_1005Metric, F.Cu at (162.4, 137.0)
- added C15: 100nF, Capacitor_SMD:C_0402_1005Metric, F.Cu at (164.2, 140.3)
- added P1: USB_C_Plug_USB2.0, Connector_USB:USB_C_Plug_Molex_105444, F.Cu at (133.4, 133.5)
- added U2: LSM6DS3TR-C, ST:QFN_S3TR-C_STM, F.Cu at (165.0, 137.5)
- added Y2: 32.768khz, Crystal:Crystal_SMD_2016-4Pin_2.0x1.6mm, F.Cu at (168.5, 125.2)
Connections:
- U1 pad 16: unconnected-(U1-P2.05-Pad16) -> /IMU_CS
- U1 pad 17: unconnected-(U1-P2.06-Pad17) -> /IMU_CLK
- U1 pad 19: unconnected-(U1-P2.08-Pad19) -> /IMU_MOSI
- U1 pad 20: unconnected-(U1-P2.09-Pad20) -> /IMU_MISO
- U1 pad 23: unconnected-(U1-P0.00-Pad23) -> Net-(U1-P0.00)
- U1 pad 24: unconnected-(U1-P0.01-Pad24) -> Net-(U1-P0.01)
Routing:
- net /IMU_MOSI: track 0.00 -> 11.1 mm, vias 0 -> 2
- net /IMU_CLK: track 0.00 -> 10.8 mm, vias 0 -> 2
- net /IMU_CS: track 0.00 -> 10.7 mm, vias 0 -> 2
- net /IMU_MISO: track 0.00 -> 10.2 mm, vias 0 -> 2
- net GND: track 20.3 -> 23.2 mm, vias 13 -> 14
- net Net-(U1-P0.00): track 0.00 -> 2.94 mm
- net Net-(U1-P0.01): track 0.00 -> 2.46 mm
- net /3v3: track 0.00 -> 2.31 mm

Commit message: RF, ESD, tiny
Parts:
- removed P1: USB_C_Plug_USB2.0, Connector_USB:USB_C_Plug_Molex_105444
- added C16: 1uF, Capacitor_SMD:C_0201_0603Metric, F.Cu at (193.2, 147.0)
- added C17: 2.2uF, Capacitor_SMD:C_0603_1608Metric, F.Cu at (190.5, 147.4)
- added C18: 10uF, Capacitor_SMD:C_0603_1608Metric, F.Cu at (191.2, 145.8)
- added C19: 10uF, Capacitor_SMD:C_0603_1608Metric, F.Cu at (189.2, 151.1)
- added C20: 10uF, Capacitor_SMD:C_0603_1608Metric, F.Cu at (188.6, 154.1)
- added C21: 100nF, Capacitor_SMD:C_0201_0603Metric, F.Cu at (165.9, 127.2)
- added J1: Pin1, Connector_Wire:SolderWirePad_1x01_SMD_1.5x3mm, F.Cu at (162.7, 146.1)
- added J2: Pin2, Connector_Wire:SolderWirePad_1x01_SMD_1.5x3mm, F.Cu at (165.8, 146.1)
- added J3: USB_C_Receptacle_USB2.0_14P, Connector_USB:USB_C_Receptacle_HRO_TYPE-C-31-M-12, F.Cu at (154.2, 126.9)
- added J4: Pin3, Connector_Wire:SolderWirePad_1x01_SMD_1.5x3mm, F.Cu at (168.8, 146.1)
- added J5: Pin, Connector_Wire:SolderWirePad_1x01_SMD_1.5x3mm, F.Cu at (203.5, 125.0)
- added J6: Pin, Connector_Wire:SolderWirePad_1x01_SMD_1.5x3mm, F.Cu at (203.5, 122.7)
- added J7: Pin, Connector_Wire:SolderWirePad_1x01_SMD_1.5x3mm, F.Cu at (203.5, 127.3)
- added J8: Conn_01x02_Pin, ST:Inverted_F_Antenna_2.4Ghz_1.0mmPCB_TI_CC2430DB.pretty, F.Cu at (152.2, 110.5)
- added L5: 2.2uH, ST:IND_TAIYO_LBM2016_TAY, F.Cu at (187.2, 151.8)
- added R2: 1.5k, Resistor_SMD:R_0201_0603Metric, F.Cu at (195.6, 148.4)
- added R3: 5.1k, Resistor_SMD:R_0201_0603Metric, F.Cu at (160.3, 128.7)
- added R4: 5.1k, Resistor_SMD:R_0201_0603Metric, F.Cu at (160.3, 125.7)
- added U3: nPM1100-QDXX, Package_DFN_QFN:QFN-24-1EP_4x4mm_P0.5mm_EP2.6x2.6mm_ThermalVias, F.Cu at (192.6, 150.8)
- added U4: USBLC6-2SC6, Package_TO_SOT_SMD:SOT-23-6, F.Cu at (163.1, 127.2)
- moved C13 45.9 mm to (160.6, 164.3), turned to -90 degrees
- moved Y1 44.8 mm to (165.6, 167.8), turned to 90 degrees
- moved L4 44.4 mm to (161.8, 164.0), turned to 180 degrees
- moved L2 43.1 mm to (170.9, 169.7), turned to 180 degrees
- moved C3 43.0 mm to (167.7, 167.8), turned to -90 degrees
- moved C12 43.0 mm to (165.0, 165.7), turned to 180 degrees
- moved C11 42.9 mm to (162.9, 163.7), turned to 90 degrees
- moved C15 42.4 mm to (169.1, 168.2), turned to -90 degrees
- moved L3 42.1 mm to (164.1, 164.0), turned to 180 degrees
- moved FB1 41.9 mm to (169.9, 168.2), turned to -90 degrees
- moved C10 41.5 mm to (165.6, 164.8), turned to 0 degrees
- moved C14 41.3 mm to (170.6, 168.2), turned to -90 degrees
- moved L1 40.7 mm to (165.6, 164.0), turned to 180 degrees
- moved C8 40.3 mm to (172.1, 168.2), turned to -90 degrees
- moved C4 39.9 mm to (172.9, 168.2), turned to -90 degrees
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- renumbered C14 to C1, C6 to C12, C12 to C13, C7 to C14, C8 to C15, C15 to C2, C1 to C3, C2 to C4, C3 to C5, C4 to C6, C5 to C7, C9 to C8, C13 to C9, L2 to L1, L1 to L2, U2 to U1, U1 to U2
Connections:
- C13 pad 1: GND -> /RF
- C3 pad 1: /VDD_MCU -> /3v3
- C4 pad 1: /VDD_MCU -> /3v3
- C5 pad 1: /VDD_MCU -> /3v3
- C6 pad 1: /VDD_MCU -> /3v3
- C7 pad 1: /VDD_MCU -> /3v3
- L4 pad 2: GND -> /RF
- U2 pad 10: /VDD_MCU -> /3v3
- U2 pad 22: /VDD_MCU -> /3v3
- U2 pad 36: /VDD_MCU -> /3v3
- U2 pad 47: /VDD_MCU -> /3v3
- U2 pad 48: /VDD_MCU -> /3v3
Routing:
- net /3v3: track 2.31 -> 23.5 mm
- net /VSYS: track 0.00 -> 14.2 mm, vias 0 -> 3
- net /USB_5V: track 0.00 -> 12.7 mm, vias 0 -> 2
- net /IMU_MOSI: track 11.1 -> 2.22 mm
- net /IMU_CLK: track 10.8 -> 2.11 mm
- net /IMU_CS: track 10.7 -> 2.27 mm
- net /IMU_MISO: track 10.2 -> 2.02 mm, vias 2 -> 1
- net /USB_D-: track 0.00 -> 6.28 mm
- net /VDD_MCU: track 6.09 -> 0.00 mm
- net /USB_D+: track 0.00 -> 5.69 mm
- net GND: track 23.2 -> 27.9 mm, vias 14 -> 51
- net Net-(J1-Pin_1): track 0.00 -> 4.04 mm, vias 0 -> 2
- net Net-(U3-SW): track 0.00 -> 3.46 mm
- net /SWDIO: track 0.00 -> 3.28 mm, vias 0 -> 2
- net Net-(J3-CC2): track 0.00 -> 1.69 mm
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Other:
- outline, holes or cut-outs redrawn
- board text added: "- Y"
- board text added: "-X"
- board text added: "-Z"
- board text added: "Iiimote"
- board text added: "v1.0"

Commit message: routeds
Parts:
- L5: footprint ST:IND_TAIYO_LBM2016_TAY -> ST:APH201610C2R2MP01
- Y2: footprint Crystal:Crystal_SMD_2016-4Pin_2.0x1.6mm -> Crystal:Crystal_SMD_2012-2Pin_2.0x1.2mm
- moved Y1 44.6 mm to (153.3, 124.9), turned to 0 degrees
- moved C13 44.6 mm to (156.7, 120.0), turned to 180 degrees
- moved L2 44.0 mm to (151.4, 130.2), turned to 90 degrees
- moved C3 43.2 mm to (153.3, 127.0), turned to 180 degrees
- moved L4 43.2 mm to (157.1, 121.1), turned to 90 degrees
- moved C15 42.9 mm to (152.9, 128.4), turned to 180 degrees
- moved FB1 42.5 mm to (152.9, 129.2), turned to 180 degrees
- moved C12 42.5 mm to (155.4, 124.3), turned to 90 degrees
- moved C14 42.1 mm to (152.9, 129.9), turned to 180 degrees
- moved C11 41.8 mm to (157.4, 122.2), turned to 0 degrees
- moved R2 41.6 mm to (166.1, 119.2), turned to 180 degrees
- moved C8 41.4 mm to (152.9, 131.4), turned to 180 degrees
- moved G 41.3 mm to (163.6, 138.1), turned to 0 degrees
- moved L3 41.2 mm to (157.1, 123.4), turned to 90 degrees
- moved C4 41.1 mm to (152.9, 132.2), turned to 180 degrees
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- renumbered J1 to +, J2 to -, J5 to CL, J7 to G, J6 to IO, J4 to TS
Connections:
- Y2 pad 2: GND -> Net-(U2-P0.00)
Routing:
- net /3v3: track 23.5 -> 57.7 mm, vias 0 -> 5
- net /SWDCLK: track 0.00 -> 32.3 mm, vias 0 -> 2
- net /SWDIO: track 3.28 -> 33.5 mm
- net /NTC: track 0.00 -> 19.9 mm, vias 0 -> 4
- net Net-(J1-Pin_1): track 4.04 -> 22.6 mm
- net /SYS_D+: track 0.00 -> 11.3 mm, vias 0 -> 2
- net /SYS_D-: track 0.00 -> 11.2 mm, vias 0 -> 2
- net /USB_5V: track 12.7 -> 23.7 mm
- net GND: track 27.9 -> 19.7 mm, vias 51 -> 74
- net /RF: track 0.00 -> 7.54 mm
- net /IMU_CS: track 2.27 -> 8.52 mm
- net /IMU_MOSI: track 2.22 -> 7.15 mm
- net /IMU_MISO: track 2.02 -> 5.91 mm, vias 1 -> 2
- net /IMU_CLK: track 2.11 -> 4.57 mm
- net Net-(U2-P0.00): track 2.94 -> 2.17 mm
Other:
- board size 30 x 39.5 mm -> 30 x 30 mm
- board text added: "X"
- board text added: "Z"
- board text removed: "-X"
- board text removed: "-Z"
