File: imu-gc.kicad_pcb (KiCad board)
At the start: 2 copper layers, 30 x 30 mm, 45 parts, among them J3 USB_C_Receptacle_USB2.0_14P, J8 Conn_01x02_Pin, U1 LSM6DS3TR-C, U2 nRF54L15-QFXX, U3 nPM1100-QDXX, U4 USBLC6-2SC6, Y1 32Mhz, Y2 32.768khz

Commit message: gen'd bom
Routing:
- net /3v3: vias 5 -> 6
Other:
- board text added: "Iiiriomote"
- board text removed: "Iiimote"

Commit message: boms
Other:
- copper layers 2 -> 4
Changed lines of the file:
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@@
 	(layers
 		(0 "F.Cu" signal)
+		(4 "In1.Cu" signal)
+		(6 "In2.Cu" signal)
 		(2 "B.Cu" signal)
 		(9 "F.Adhes" user "F.Adhesive")
@@
 			)
 			(layer "dielectric 1"
+				(type "prepreg")
+				(thickness 0.1)
+				(material "FR4")
+				(epsilon_r 4.5)
+				(loss_tangent 0.02)
+			)
+			(layer "In1.Cu"
+				(type "copper")
+				(thickness 0.035)
+			)
+			(layer "dielectric 2"
 				(type "core")
-				(thickness 1.51)
+				(thickness 1.24)
+				(material "FR4")
+				(epsilon_r 4.5)
+				(loss_tangent 0.02)
+			)
+			(layer "In2.Cu"
+				(type "copper")
+				(thickness 0.035)
+			)
+			(layer "dielectric 3"
+				(type "prepreg")
+				(thickness 0.1)
 				(material "FR4")
 				(epsilon_r 4.5)
@@
 		(capping no)
 		(filling no)
+		(zone_defaults)
 		(pcbplotparams
 			(layerselection 0x00000000_00000000_55555555_5755f5ff)

Commit message: jlc les goo
Parts:
- C9: footprint Capacitor_SMD:C_0402_1005Metric -> Capacitor_SMD:C_0201_0603Metric
- moved J3 1.03 mm to (174.2, 135.8)
- moved C9 0.21 mm to (158.6, 125.7)
- renumbered + to J1, - to J2, TS to J4, CL to J5, IO to J6, G to J7
Routing:
- net /USB_D+: track 5.69 -> 7.45 mm
- net GND: track 19.7 -> 20.9 mm, vias 74 -> 75
- net /USB_D-: track 6.28 -> 7.31 mm
- net /USB_5V: track 23.7 -> 24.8 mm
- net Net-(J3-CC2): track 1.69 -> 2.72 mm
- net Net-(J3-CC1): track 1.69 -> 2.72 mm
- added copper zone on In1.Cu, net GND
- added copper zone on In2.Cu, net GND

Commit message: bc
Parts:
- added B: Pin, Connector_Wire:SolderWirePad_1x01_SMD_1x2mm, F.Cu at (178.0, 123.6)
- added G: Pin, Connector_Wire:SolderWirePad_1x01_SMD_1x2mm, F.Cu at (174.5, 121.0)
- added R5: 4.7k, Resistor_SMD:R_0201_0603Metric, F.Cu at (160.9, 133.3)
- renumbered J1 to +, J2 to -, J5 to CL, J7 to G, J6 to IO, J4 to TS
Connections:
- U2 pad 13: unconnected-(U2-P2.02-Pad13) -> Net-(J10-Pin_1)
Routing:
- net Net-(J10-Pin_1): track 0.00 -> 31.9 mm, vias 0 -> 2
- net /USB_D+: track 7.45 -> 6.72 mm
- net /3v3: track 57.7 -> 58.3 mm
