File: imu-gc.kicad_sch (KiCad schematic)
At the start: 21 parts, among them U1 nRF54L15-QFXX, Y1 32Mhz

Commit message: typ l
Parts:
- C10: renamed from C8; footprint Capacitor_SMD:C_0402_1005Metric -> Capacitor_SMD:C_0201_0603Metric
- C11: renamed from C9; footprint Capacitor_SMD:C_0402_1005Metric -> Capacitor_SMD:C_0201_0603Metric
- C12: renamed from C11; footprint Capacitor_SMD:C_0402_1005Metric -> Capacitor_SMD:C_0201_0603Metric
- L2: renamed from L1; footprint Inductor_SMD:L_0402_1005Metric -> Inductor_SMD:L_0201_0603Metric
- L3, L4: footprint Inductor_SMD:L_0402_1005Metric -> Inductor_SMD:L_0201_0603Metric
- renumbered C7 to C13, C10 to C6, C12 to C7, C13 to C8, C6 to C9, L2 to L1
Changed lines of the file:
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@@
 		(dnp no)
 		(fields_autoplaced yes)
-		(property "Reference" "C6"
+		(property "Reference" "C9"
 			(at 177.8 66.0399 0)
 			(show_name no)
@@
 			(project "imu-gc"
 				(path "/34e09bf3-607e-4d30-9b2e-53b693860bcd"
-					(reference "C6")
+					(reference "C9")
 					(unit 1)
 				)
@@
 		(in_pos_files yes)
 		(dnp no)
-		(property "Reference" "C10"
+		(property "Reference" "C6"
 			(at 199.39 58.928 0)
 			(show_name no)
@@
 			(project "imu-gc"
 				(path "/34e09bf3-607e-4d30-9b2e-53b693860bcd"
-					(reference "C10")
+					(reference "C6")
 					(unit 1)
 				)
@@
 		(dnp no)
 		(fields_autoplaced yes)
-		(property "Reference" "#PWR014"
+		(property "Reference" "#PWR09"
 			(at 218.44 69.85 0)
 			(hide yes)
@@
 			(project "imu-gc"
 				(path "/34e09bf3-607e-4d30-9b2e-53b693860bcd"
-					(reference "#PWR014")
+					(reference "#PWR09")
 					(unit 1)
 				)
@@
 		(dnp no)
 		(fields_autoplaced yes)
-		(property "Reference" "C7"
+		(property "Reference" "C13"
 			(at 177.8 154.9399 0)
 			(show_name no)
@@
 			(project "imu-gc"
 				(path "/34e09bf3-607e-4d30-9b2e-53b693860bcd"
-					(reference "C7")
+					(reference "C13")
 					(unit 1)
 				)
@@
 		(dnp no)
 		(fields_autoplaced yes)
-		(property "Reference" "#PWR011"
+		(property "Reference" "#PWR07"
 			(at 195.58 69.85 0)
 			(hide yes)
@@
 			(project "imu-gc"
 				(path "/34e09bf3-607e-4d30-9b2e-53b693860bcd"
-					(reference "#PWR011")
+					(reference "#PWR07")
 					(unit 1)
 				)
@@
 		(dnp no)
 		(fields_autoplaced yes)
-		(property "Reference" "#PWR010"
+		(property "Reference" "#PWR012"
 			(at 193.04 115.57 0)
 			(hide yes)
@@
 			(project "imu-gc"
 				(path "/34e09bf3-607e-4d30-9b2e-53b693860bcd"
-					(reference "#PWR010")
+					(reference "#PWR012")
 					(unit 1)
 				)
@@
 		(dnp no)
 		(fields_autoplaced yes)
-		(property "Reference" "#PWR07"
+		(property "Reference" "#PWR014"
 			(at 142.24 166.37 0)
 			(hide yes)
@@
 			(project "imu-gc"
 				(path "/34e09bf3-607e-4d30-9b2e-53b693860bcd"
-					(reference "#PWR07")
+					(reference "#PWR014")
 					(unit 1)
 				)
@@
 		(dnp no)
 		(fields_autoplaced yes)
-		(property "Reference" "C11"
+		(property "Reference" "C12"
 			(at 209.55 102.8699 0)
 			(show_name no)
@@
 			)
 		)
-		(property "Footprint" "Capacitor_SMD:C_0402_1005Metric"
+		(property "Footprint" "Capacitor_SMD:C_0201_0603Metric"
 			(at 206.7052 107.95 0)
 			(hide yes)
@@
 			(project "imu-gc"
 				(path "/34e09bf3-607e-4d30-9b2e-53b693860bcd"
-					(reference "C11")
+					(reference "C12")
 					(unit 1)
 				)
@@
 		(dnp no)
 		(fields_autoplaced yes)
-		(property "Reference" "#PWR09"
+		(property "Reference" "#PWR011"
 			(at 180.34 115.57 0)
 			(hide yes)
@@
 			(project "imu-gc"
 				(path "/34e09bf3-607e-4d30-9b2e-53b693860bcd"
-					(reference "#PWR09")
+					(reference "#PWR011")
 					(unit 1)
 				)
@@
 			)
 		)
-		(property "Footprint" "Inductor_SMD:L_0402_1005Metric"
+		(property "Footprint" "Inductor_SMD:L_0201_0603Metric"
 			(at 198.12 100.33 0)
 			(hide yes)
@@
 		(in_pos_files yes)
 		(dnp no)
-		(property "Reference" "#PWR06"
+		(property "Reference" "#PWR05"
 			(at 138.43 45.72 0)
 			(hide yes)
@@
 			(project "imu-gc"
 				(path "/34e09bf3-607e-4d30-9b2e-53b693860bcd"
-					(reference "#PWR06")
+					(reference "#PWR05")
 					(unit 1)
 				)
@@
 		(dnp no)
 		(fields_autoplaced yes)
-		(property "Reference" "#PWR03"
+		(property "Reference" "#PWR06"
 			(at 107.95 63.5 0)
 			(hide yes)
@@
 			(project "imu-gc"
 				(path "/34e09bf3-607e-4d30-9b2e-53b693860bcd"
-					(reference "#PWR03")
+					(reference "#PWR06")
 					(unit 1)
 				)
@@
 		(dnp no)
 		(fields_autoplaced yes)
-		(property "Reference" "L1"
+		(property "Reference" "L2"
 			(at 175.26 95.25 90)
 			(show_name no)
@@
 			)
 		)
-		(property "Footprint" "Inductor_SMD:L_0402_1005Metric"
+		(property "Footprint" "Inductor_SMD:L_0201_0603Metric"
 			(at 175.26 100.33 0)
 			(hide yes)
@@
 			(project "imu-gc"
 				(path "/34e09bf3-607e-4d30-9b2e-53b693860bcd"
-					(reference "L1")
+					(reference "L2")
 					(unit 1)
 				)
@@
 		(dnp no)
 		(fields_autoplaced yes)
-		(property "Reference" "#PWR012"
+		(property "Reference" "#PWR013"
 			(at 205.74 115.57 0)
 			(hide yes)
@@
 			(project "imu-gc"
 				(path "/34e09bf3-607e-4d30-9b2e-53b693860bcd"
-					(reference "#PWR012")
+					(reference "#PWR013")
 					(unit 1)
 				)
@@
 		(dnp no)
 		(fields_autoplaced yes)
-		(property "Reference" "L2"
+		(property "Reference" "L1"
 			(at 177.8 58.4199 0)
 			(show_name no)
@@
 			(project "imu-gc"
 				(path "/34e09bf3-607e-4d30-9b2e-53b693860bcd"
-					(reference "L2")
+					(reference "L1")
 					(unit 1)
 				)
@@
 		(in_pos_files yes)
 		(dnp no)
-		(property "Reference" "C12"
+		(property "Reference" "C7"
 			(at 210.566 58.928 0)
 			(show_name no)
@@
 			(project "imu-gc"
 				(path "/34e09bf3-607e-4d30-9b2e-53b693860bcd"
-					(reference "C12")
+					(reference "C7")
 					(unit 1)
 				)
@@
 		(dnp no)
 		(fields_autoplaced yes)
-		(property "Reference" "#PWR013"
+		(property "Reference" "#PWR08"
 			(at 207.01 69.85 0)
 			(hide yes)
@@
 			(project "imu-gc"
 				(path "/34e09bf3-607e-4d30-9b2e-53b693860bcd"
-					(reference "#PWR013")
+					(reference "#PWR08")
 					(unit 1)
 				)
@@
 			)
 		)
-		(property "Footprint" "Inductor_SMD:L_0402_1005Metric"
+		(property "Footprint" "Inductor_SMD:L_0201_0603Metric"
 			(at 185.42 100.33 0)
 			(hide yes)
@@
 		(dnp no)
 		(fields_autoplaced yes)
-		(property "Reference" "C8"
+		(property "Reference" "C10"
 			(at 184.15 102.8699 0)
 			(show_name no)
@@
 			)
 		)
-		(property "Footprint" "Capacitor_SMD:C_0402_1005Metric"
+		(property "Footprint" "Capacitor_SMD:C_0201_0603Metric"
 			(at 181.3052 107.95 0)
 			(hide yes)
@@
 			(project "imu-gc"
 				(path "/34e09bf3-607e-4d30-9b2e-53b693860bcd"
-					(reference "C8")
+					(reference "C10")
 					(unit 1)
 				)
@@
 		(in_pos_files yes)
 		(dnp no)
-		(property "Reference" "#PWR04"
+		(property "Reference" "#PWR03"
 			(at 110.49 45.72 0)
 			(hide yes)
@@
 			(project "imu-gc"
 				(path "/34e09bf3-607e-4d30-9b2e-53b693860bcd"
-					(reference "#PWR04")
+					(reference "#PWR03")
 					(unit 1)
 				)
@@
 		(dnp no)
 		(fields_autoplaced yes)
-		(property "Reference" "#PWR08"
+		(property "Reference" "#PWR010"
 			(at 173.99 78.74 0)
 			(hide yes)
@@
 			(project "imu-gc"
 				(path "/34e09bf3-607e-4d30-9b2e-53b693860bcd"
-					(reference "#PWR08")
+					(reference "#PWR010")
 					(unit 1)
 				)
@@
 		(dnp no)
 		(fields_autoplaced yes)
-		(property "Reference" "C9"
+		(property "Reference" "C11"
 			(at 196.85 102.8699 0)
 			(show_name no)
@@
 			)
 		)
-		(property "Footprint" "Capacitor_SMD:C_0402_1005Metric"
+		(property "Footprint" "Capacitor_SMD:C_0201_0603Metric"
 			(at 194.0052 107.95 0)
 			(hide yes)
@@
 			(project "imu-gc"
 				(path "/34e09bf3-607e-4d30-9b2e-53b693860bcd"
-					(reference "C9")
+					(reference "C11")
 					(unit 1)
 				)
@@
 		(in_pos_files yes)
 		(dnp no)
-		(property "Reference" "#PWR05"
+		(property "Reference" "#PWR04"
 			(at 124.46 45.72 0)
 			(hide yes)
@@
 			(project "imu-gc"
 				(path "/34e09bf3-607e-4d30-9b2e-53b693860bcd"
-					(reference "#PWR05")
+					(reference "#PWR04")
 					(unit 1)
 				)
@@
 		(dnp no)
 		(fields_autoplaced yes)
-		(property "Reference" "C13"
+		(property "Reference" "C8"
 			(at 222.25 57.1499 0)
 			(show_name no)
@@
 			(project "imu-gc"
 				(path "/34e09bf3-607e-4d30-9b2e-53b693860bcd"
-					(reference "C13")
-					(unit 1)
-				)
+					(reference "C8")
+					(unit 1)
+				)

Commit message: Atennas? RF for sures
Connections:
- net RF is gone; now on net GND: C12.1, L4.2
Changed lines of the file:
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@@
 	(wire
 		(pts
-			(xy 201.93 100.33) (xy 210.82 100.33)
+			(xy 201.93 100.33) (xy 218.44 100.33)
+		)
+		(stroke
+			(width 0)
+			(type default)
+		)
+	)
+	(wire
+		(pts
+			(xy 218.44 100.33) (xy 218.44 109.22)
 		)
 		(stroke
@@
 					(unit 1)
 				)
+			)
+		)
+	)
+	(symbol
+		(lib_id "power:GND")
+		(at 218.44 109.22 0)
+		(unit 1)
+		(body_style 1)
+		(exclude_from_sim no)
+		(in_bom yes)
+		(on_board yes)
+		(in_pos_files yes)
+		(dnp no)
+		(fields_autoplaced yes)
+		(property "Reference" "#PWR015"
+			(at 218.44 115.57 0)
+			(hide yes)
+			(show_name no)
+			(do_not_autoplace no)
+			(effects
+				(font
+					(size 1.27 1.27)
+				)
+			)
+		)
+		(property "Value" "GND"
+			(at 218.44 114.3 0)
+			(show_name no)
+			(do_not_autoplace no)
+			(effects
+				(font
+					(size 1.27 1.27)
+				)
+			)
+		)
+		(property "Footprint" ""
+			(at 218.44 109.22 0)
+			(hide yes)
+			(show_name no)
+			(do_not_autoplace no)
+			(effects
+				(font
+					(size 1.27 1.27)
+				)
+			)
+		)
+		(property "Datasheet" ""
+			(at 218.44 109.22 0)
+			(hide yes)
+			(show_name no)
+			(do_not_autoplace no)
+			(effects
+				(font
+					(size 1.27 1.27)
+				)
+			)
+		)
+		(property "Description" "Power symbol creates a global label with name \"GND\" , ground"
+			(at 218.44 109.22 0)
+			(hide yes)
+			(show_name no)
+			(do_not_autoplace no)
+			(effects
+				(font
+					(size 1.27 1.27)
+				)
+			)
+		)
+		(pin "1"
+		)
+		(instances
+			(project "imu-gc"
+				(path "/34e09bf3-607e-4d30-9b2e-53b693860bcd"
+					(reference "#PWR015")
+					(unit 1)
+				)

Commit message: typ finsihed. yeygit add -A
Parts:
- C1, C2, C4, C5: value 1000nF -> 100nF; footprint Capacitor_SMD:C_0402_1005Metric -> Capacitor_SMD:C_0201_0603Metric
- C3: value 1000nF -> 10uF
- C6, C7, C8, C9: footprint Capacitor_SMD:C_0402_1005Metric -> Capacitor_SMD:C_0201_0603Metric
- FB1: footprint Inductor_SMD:L_0402_1005Metric -> Inductor_SMD:L_0201_0603Metric
- L1: footprint Inductor_SMD:L_0402_1005Metric -> Inductor_SMD:L_0603_1608Metric
- R1: footprint Resistor_SMD:R_0402_1005Metric -> Resistor_SMD:R_0201_0603Metric
Connections:
- net GND: now also C13.2
Changed lines of the file:
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@@
 			)
 		)
-		(property "Footprint" "Capacitor_SMD:C_0402_1005Metric"
+		(property "Footprint" "Capacitor_SMD:C_0201_0603Metric"
 			(at 174.9552 71.12 0)
 			(hide yes)
@@
 			)
 		)
-		(property "Footprint" "Capacitor_SMD:C_0402_1005Metric"
+		(property "Footprint" "Capacitor_SMD:C_0201_0603Metric"
 			(at 196.5452 62.23 0)
 			(hide yes)
@@
 			)
 		)
-		(property "Value" "1000nF"
+		(property "Value" "100nF"
 			(at 128.27 35.5599 0)
 			(show_name no)
@@
 			)
 		)
-		(property "Footprint" "Capacitor_SMD:C_0402_1005Metric"
+		(property "Footprint" "Capacitor_SMD:C_0201_0603Metric"
 			(at 125.4252 38.1 0)
 			(hide yes)
@@
 			)
 		)
-		(property "Value" "1000nF"
+		(property "Value" "10uF"
 			(at 114.3 35.5599 0)
 			(show_name no)
@@
 	(symbol
 		(lib_id "power:GND")
+		(at 173.99 160.02 0)
+		(unit 1)
+		(body_style 1)
+		(exclude_from_sim no)
+		(in_bom yes)
+		(on_board yes)
+		(in_pos_files yes)
+		(dnp no)
+		(fields_autoplaced yes)
+		(property "Reference" "#PWR016"
+			(at 173.99 166.37 0)
+			(hide yes)
+			(show_name no)
+			(do_not_autoplace no)
+			(effects
+				(font
+					(size 1.27 1.27)
+				)
+			)
+		)
+		(property "Value" "GND"
+			(at 173.99 165.1 0)
+			(show_name no)
+			(do_not_autoplace no)
+			(effects
+				(font
+					(size 1.27 1.27)
+				)
+			)
+		)
+		(property "Footprint" ""
+			(at 173.99 160.02 0)
+			(hide yes)
+			(show_name no)
+			(do_not_autoplace no)
+			(effects
+				(font
+					(size 1.27 1.27)
+				)
+			)
+		)
+		(property "Datasheet" ""
+			(at 173.99 160.02 0)
+			(hide yes)
+			(show_name no)
+			(do_not_autoplace no)
+			(effects
+				(font
+					(size 1.27 1.27)
+				)
+			)
+		)
+		(property "Description" "Power symbol creates a global label with name \"GND\" , ground"
+			(at 173.99 160.02 0)
+			(hide yes)
+			(show_name no)
+			(do_not_autoplace no)
+			(effects
+				(font
+					(size 1.27 1.27)
+				)
+			)
+		)
+		(pin "1"
+		)
+		(instances
+			(project "imu-gc"
+				(path "/34e09bf3-607e-4d30-9b2e-53b693860bcd"
+					(reference "#PWR016")
+					(unit 1)
+				)
+			)
+		)
+	)
+	(symbol
+		(lib_id "power:GND")
 		(at 180.34 109.22 0)
 		(unit 1)
@@
 			)
 		)
-		(property "Value" "1000nF"
+		(property "Value" "100nF"
 			(at 86.36 35.5599 0)
 			(show_name no)
@@
 			)
 		)
-		(property "Footprint" "Capacitor_SMD:C_0402_1005Metric"
+		(property "Footprint" "Capacitor_SMD:C_0201_0603Metric"
 			(at 83.5152 38.1 0)
 			(hide yes)
@@
 			)
 		)
-		(property "Value" "1000nF"
+		(property "Value" "100nF"
 			(at 100.33 35.5599 0)
 			(show_name no)
@@
 			)
 		)
-		(property "Footprint" "Capacitor_SMD:C_0402_1005Metric"
+		(property "Footprint" "Capacitor_SMD:C_0201_0603Metric"
 			(at 97.4852 38.1 0)
 			(hide yes)
@@
 			)
 		)
-		(property "Footprint" "Resistor_SMD:R_0402_1005Metric"
+		(property "Footprint" "Resistor_SMD:R_0201_0603Metric"
 			(at 179.07 145.288 90)
 			(hide yes)
@@
 			)
 		)
-		(property "Footprint" "Inductor_SMD:L_0402_1005Metric"
+		(property "Footprint" "Inductor_SMD:L_0201_0603Metric"
 			(at 182.372 58.42 90)
 			(hide yes)
@@
 			)
 		)
-		(property "Footprint" "Inductor_SMD:L_0402_1005Metric"
+		(property "Footprint" "Inductor_SMD:L_0603_1608Metric"
 			(at 176.53 59.69 0)
 			(hide yes)
@@
 			)
 		)
-		(property "Footprint" "Capacitor_SMD:C_0402_1005Metric"
+		(property "Footprint" "Capacitor_SMD:C_0201_0603Metric"
 			(at 207.9752 62.23 0)
 			(hide yes)
@@
 			)
 		)
-		(property "Value" "1000nF"
+		(property "Value" "100nF"
 			(at 142.24 35.5599 0)
 			(show_name no)
@@
 			)
 		)
-		(property "Footprint" "Capacitor_SMD:C_0402_1005Metric"
+		(property "Footprint" "Capacitor_SMD:C_0201_0603Metric"
 			(at 139.3952 38.1 0)
 			(hide yes)
@@
 			)
 		)
-		(property "Footprint" "Capacitor_SMD:C_0402_1005Metric"
+		(property "Footprint" "Capacitor_SMD:C_0201_0603Metric"
 			(at 219.4052 62.23 0)
 			(hide yes)

Commit message: IMU ok, power startd
Parts:
- added C14, C15: 100nF, Capacitor_SMD:C_0402_1005Metric, symbol Device:C
- added U2: LSM6DS3TR-C, ST:QFN_S3TR-C_STM, symbol ST LSM6DS3TR-C:LSM6DS3TR-C
- added Y2: 32.768khz, Crystal:Crystal_SMD_2016-4Pin_2.0x1.6mm, symbol Device:Crystal_GND24
Connections:
- net GND: now also C14.2, C15.2, U2.2 (SDx), U2.3 (SCx), U2.6 (GND), U2.7 (GND), Y2.2 (G), Y2.4 (G)
- net IMU_CS: now reaches U1.16 (P2.05)
- net IMU_CS: now also U2.12 (CS)
- net IMU_CLK: now reaches U1.17 (P2.06)
- net IMU_CLK: now also U2.13 (SCL)
- net IMU_MOSI: now reaches U1.19 (P2.08)
- net IMU_MOSI: now also U2.14 (SDA)
- net IMU_MISO: now reaches U1.20 (P2.09)
- net IMU_MISO: now also U2.1 (SDO/SA0)
- net at U1.23 (P0.00): now also Y2.3
- net at U1.24 (P0.01): now also Y2.1
- new net 3v3: C14.1, C15.1, U2.5 (VDDIO), U2.8 (VDD)
Other:
- added sheet Untitled Sheet (pows.kicad_sch)

Commit message: RF, ESD, tiny
Parts:
- added C16: 1uF, Capacitor_SMD:C_0201_0603Metric, symbol Device:C
- added C17: 2.2uF, Capacitor_SMD:C_0603_1608Metric, symbol Device:C
- added C18, C19, C20: 10uF, Capacitor_SMD:C_0603_1608Metric, symbol Device:C
- added C21: 100nF, Capacitor_SMD:C_0201_0603Metric, symbol Device:C
- added J1: Pin1, Connector_Wire:SolderWirePad_1x01_SMD_1.5x3mm, symbol Connector:Conn_01x01_Pin
- added J2: Pin2, Connector_Wire:SolderWirePad_1x01_SMD_1.5x3mm, symbol Connector:Conn_01x01_Pin
- added J3: USB_C_Receptacle_USB2.0_14P, Connector_USB:USB_C_Receptacle_HRO_TYPE-C-31-M-12, symbol Connector:USB_C_Receptacle_USB2.0_14P
- added J4: Pin3, Connector_Wire:SolderWirePad_1x01_SMD_1.5x3mm, symbol Connector:Conn_01x01_Pin
- added J5, J6, J7: Pin, Connector_Wire:SolderWirePad_1x01_SMD_1.5x3mm, symbol Connector:Conn_01x01_Pin
- added J8: Conn_01x02_Pin, ST:Inverted_F_Antenna_2.4Ghz_1.0mmPCB_TI_CC2430DB.pretty, symbol Connector:Conn_01x02_Pin
- added L5: 2.2uH, ST:IND_TAIYO_LBM2016_TAY, symbol Device:L
- added R2: 1.5k, Resistor_SMD:R_0201_0603Metric, symbol Device:R
- added R3, R4: 5.1k, Resistor_SMD:R_0201_0603Metric, symbol Device:R
- added U3: nPM1100-QDXX, Package_DFN_QFN:QFN-24-1EP_4x4mm_P0.5mm_EP2.6x2.6mm_ThermalVias, symbol PCM_nordic-lib-kicad-npm:nPM1100-QDXX
- added U4: USBLC6-2SC6, Package_TO_SOT_SMD:SOT-23-6, symbol Power_Protection:USBLC6-2SC6
- renumbered C14 to C1, C6 to C12, C12 to C13, C7 to C14, C8 to C15, C15 to C2, C1 to C3, C2 to C4, C3 to C5, C4 to C6, C5 to C7, C9 to C8, C13 to C9, L2 to L1, L1 to L2, U2 to U1, U1 to U2
Connections:
- net VDD_MCU is gone; now on net 3v3: C3.1, C4.1, C5.1, C6.1, C7.1, U2.10 (VDD), U2.22 (VDD), U2.36 (VDD), U2.47 (VDD), U2.48 (VDD)
- net 3v3: now also C20.1, L5.1, U3.1 (VOUTB)
- net GND: now also C16.2, C17.2, C18.2, C19.2, C20.2, C21.1, J2.1 (Pin_1), J3.A1 (GND), J3.A12 (GND), J3.B1 (GND), J3.B12 (GND), J3.SH (SHIELD), J7.1 (Pin_1), J8.2 (Pin_2), R2.2, R3.2, R4.2, U3.2 (VOUTBSET1), U3.23 (PVSS), U3.25 (AVSS), U3.3 (VOUTBSET0), U3.4 (AVSS), U4.2 (GND); no longer C13.1, L4.2
- net SWDCLK: now also J5.1 (Pin_1)
- net SWDIO: now also J6.1 (Pin_1)
- new net: J3.A5 (CC1), R4.1
- new net: L5.2, U3.22 (SW)
- new net: C16.1, J1.1 (Pin_1), U3.15 (VBAT)
- new net: C21.2, U4.5 (VBUS)
- new net: J3.B5 (CC2), R3.1
- new net: R2.1, U3.12 (ICHG)
- new net: C19.1, U3.21 (DEC)
- new net CHG: U3.8 (CHG)
- new net ERR: U3.10 (ERR)
- new net MODE: U3.7 (MODE)
- new net NTC: J4.1 (Pin_1), U3.14 (NTC)
- new net RF: C13.1, J8.1 (Pin_1), L4.2
- new net SHPACT: U3.6 (SHPACT)
- new net SHPHLD: U3.11 (SHPHLD)
- new net SYS_D+: U3.20 (D+), U4.4 (I/O2)
- new net SYS_D-: U3.19 (D-), U4.6 (I/O1)
- new net USB_5V: C17.1, J3.A4 (VBUS), J3.A9 (VBUS), J3.B4 (VBUS), J3.B9 (VBUS), U3.17 (VBUS)
- new net USB_D+: J3.A6 (D+), J3.B6 (D+), U4.3 (I/O2)
- new net USB_D-: J3.A7 (D-), J3.B7 (D-), U4.1 (I/O1)
- new net VSYS: C18.1, U3.16 (VSYS), U3.5 (ISET), U3.9 (VTERMSET)
Other:
- removed sheet Untitled Sheet

Commit message: routeds
Parts:
- L5: footprint ST:IND_TAIYO_LBM2016_TAY -> ST:APH201610C2R2MP01
- Y2: footprint Crystal:Crystal_SMD_2016-4Pin_2.0x1.6mm -> Crystal:Crystal_SMD_2012-2Pin_2.0x1.2mm; symbol Device:Crystal_GND24 -> Device:Crystal
Connections:
- net GND: no longer Y2.2 (G), Y2.4 (G)
- net at U2.23 (P0.00): now also Y2.2; no longer Y2.3
Changed lines of the file:
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@@
 	(wire
 		(pts
-			(xy 113.03 72.39) (xy 102.87 72.39)
+			(xy 113.03 72.39) (xy 99.06 72.39)
 		)
 		(stroke
@@
 	(wire
 		(pts
-			(xy 113.03 80.01) (xy 102.87 80.01)
+			(xy 113.03 80.01) (xy 99.06 80.01)
 		)
 		(stroke
@@
 	(wire
 		(pts
-			(xy 107.95 76.2) (xy 107.95 81.28)
-		)
-		(stroke
-			(width 0)
-			(type default)
-		)
-	)
-	(wire
-		(pts
 			(xy 170.18 151.13) (xy 190.5 151.13)
 		)
@@
 			)
 		)
-		(property "Footprint" "ST:IND_TAIYO_LBM2016_TAY"
+		(property "Footprint" "ST:APH201610C2R2MP01"
 			(at 81.28 67.31 0)
 			(hide yes)
@@
 	)
 	(symbol
-		(lib_id "power:GND")
-		(at 107.95 81.28 0)
-		(unit 1)
-		(body_style 1)
-		(exclude_from_sim no)
-		(in_bom yes)
-		(on_board yes)
-		(in_pos_files yes)
-		(dnp no)
-		(fields_autoplaced yes)
-		(property "Reference" "#PWR06"
-			(at 107.95 87.63 0)
-			(hide yes)
-			(show_name no)
-			(do_not_autoplace no)
-			(effects
-				(font
-					(size 1.27 1.27)
-				)
-			)
-		)
-		(property "Value" "GND"
-			(at 107.95 86.36 0)
-			(show_name no)
-			(do_not_autoplace no)
-			(effects
-				(font
-					(size 1.27 1.27)
-				)
-			)
-		)
-		(property "Footprint" ""
-			(at 107.95 81.28 0)
-			(hide yes)
-			(show_name no)
-			(do_not_autoplace no)
-			(effects
-				(font
-					(size 1.27 1.27)
-				)
-			)
-		)
-		(property "Datasheet" ""
-			(at 107.95 81.28 0)
-			(hide yes)
-			(show_name no)
-			(do_not_autoplace no)
-			(effects
-				(font
-					(size 1.27 1.27)
-				)
-			)
-		)
-		(property "Description" "Power symbol creates a global label with name \"GND\" , ground"
-			(at 107.95 81.28 0)
-			(hide yes)
-			(show_name no)
-			(do_not_autoplace no)
-			(effects
-				(font
-					(size 1.27 1.27)
-				)
-			)
-		)
-		(pin "1"
-		)
-		(instances
-			(project "imu-gc"
-				(path "/34e09bf3-607e-4d30-9b2e-53b693860bcd"
-					(reference "#PWR06")
-					(unit 1)
-				)
-			)
-		)
-	)
-	(symbol
 		(lib_id "Connector:Conn_01x01_Pin")
 		(at 195.58 151.13 180)
@@
 	)
 	(symbol
-		(lib_id "Device:Crystal_GND24")
-		(at 102.87 76.2 90)
+		(lib_id "Device:Crystal")
+		(at 99.06 76.2 90)
 		(unit 1)
 		(body_style 1)
@@
 		(fields_autoplaced yes)
 		(property "Reference" "Y2"
-			(at 97.79 74.9299 90)
+			(at 102.87 74.9299 90)
 			(show_name no)
 			(do_not_autoplace no)
@@
 					(size 1.27 1.27)
 				)
-				(justify left)
+				(justify right)
 			)
 		)
 		(property "Value" "32.768khz"
-			(at 97.79 77.4699 90)
+			(at 102.87 77.4699 90)
 			(show_name no)
 			(do_not_autoplace no)
@@
 					(size 1.27 1.27)
 				)
-				(justify left)
+				(justify right)
 			)
 		)
-		(property "Footprint" "Crystal:Crystal_SMD_2016-4Pin_2.0x1.6mm"
-			(at 102.87 76.2 0)
+		(property "Footprint" "Crystal:Crystal_SMD_2012-2Pin_2.0x1.2mm"
+			(at 99.06 76.2 0)
 			(hide yes)
 			(show_name no)
@@
 		)
 		(property "Datasheet" ""
-			(at 102.87 76.2 0)
+			(at 99.06 76.2 0)
 			(hide yes)
 			(show_name no)
@@
 			)
 		)
-		(property "Description" "Four pin crystal, GND on pins 2 and 4"
-			(at 102.87 76.2 0)
+		(property "Description" "Two pin crystal"
+			(at 99.06 76.2 0)
 			(hide yes)
 			(show_name no)
@@
 		)
 		(property private "KLC_S3.3" "The rectangle is not a symbol body but a graphical element"
-			(at 115.57 76.2 0)
+			(at 111.76 76.2 0)
 			(hide yes)
 			(show_name yes)
@@
 		)
 		(property private "KLC_S4.1" "Some pins are on 50mil grid to make the symbol small"
-			(at 118.11 76.2 0)
+			(at 114.3 76.2 0)
 			(hide yes)
 			(show_name yes)
@@
 			)
 		)
-		(pin "3"
-		)
 		(pin "2"
 		)
-		(pin "4"
-		)
 		(pin "1"

Commit message: jlc les goo
Parts:
- C9: footprint Capacitor_SMD:C_0402_1005Metric -> Capacitor_SMD:C_0201_0603Metric
Changed lines of the file:
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@@
 			)
 		)
-		(property "Footprint" "Capacitor_SMD:C_0402_1005Metric"
+		(property "Footprint" "Capacitor_SMD:C_0201_0603Metric"
 			(at 174.9552 160.02 0)
 			(hide yes)

Commit message: bc
Parts:
- added J10, J9: Pin, Connector_Wire:SolderWirePad_1x01_SMD_1x2mm, symbol Connector:Conn_01x01_Pin
- added R5: 4.7k, Resistor_SMD:R_0201_0603Metric, symbol Device:R
Connections:
- net 3v3: now also R5.1
- net GND: now also J9.1 (Pin_1)
- net at U2.13 (P2.02): now also J10.1 (Pin_1), R5.2
